File: Eagle/rfid_accessctl.brd (EAGLE design)
At the start: 50 x 40 mm, 27 parts, among them Q1 IRLL014

Commit message: Final updates, as per mfr
Parts:
- moved RFID_CONN 3.81 mm to (16.5, 2.54)
Routing:
- net RFID_SDA: track 34.7 -> 38.5 mm
- net RFID_SCK: track 18.4 -> 22.2 mm
- net RFID_RST: track 24.6 -> 28.4 mm
- net RFID_MOSI: track 13.8 -> 17.6 mm
- net RFID_MISO: track 16.8 -> 20.6 mm
- net VCC: track 114.0 -> 116.3 mm
Other:
- board text added: "Access Controller"
- board text added: "V_3.3"
- board text added: "V_EXT"
- board text added: "v1.2"
- board text removed: "Access Controller V1.2"
Changed lines of the file:
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@@
 <?xml version="1.0" encoding="utf-8"?>
 <!DOCTYPE eagle SYSTEM "eagle.dtd">
-<eagle version="7.6.0">
+<eagle version="7.5.0">
 <drawing>
 <settings>
@@
 <text x="46.101" y="13.081" size="1.27" layer="21" font="vector" ratio="15" rot="R180">Di</text>
 <text x="43.561" y="8.509" size="1.778" layer="21" font="vector" ratio="15" rot="R90">LED</text>
-<text x="17.653" y="2.794" size="1.77" layer="21" font="vector" ratio="15">RC522 RFID</text>
-<text x="35.052" y="9.144" size="1.27" layer="21" font="vector" ratio="15" rot="R90">VCC</text>
-<text x="17.145" y="9.144" size="1.27" layer="21" font="vector" ratio="15" rot="R90">SDA</text>
-<text x="19.685" y="9.271" size="1.27" layer="21" font="vector" ratio="15" rot="R90">SCK</text>
-<text x="22.098" y="9.398" size="1.27" layer="21" font="vector" ratio="15" rot="R90">MOSI</text>
-<text x="24.765" y="9.271" size="1.27" layer="21" font="vector" ratio="15" rot="R90">MISO</text>
-<text x="29.845" y="9.398" size="1.27" layer="21" font="vector" ratio="15" rot="R90">GND</text>
-<text x="32.385" y="9.271" size="1.27" layer="21" font="vector" ratio="15" rot="R90">RST</text>
-<text x="27.178" y="9.271" size="1.27" layer="21" font="vector" ratio="15" rot="R90">IRQ</text>
+<text x="17.653" y="12.954" size="1.77" layer="21" font="vector" ratio="15">RC522 RFID</text>
+<text x="35.052" y="4.064" size="1.27" layer="21" font="vector" ratio="15" rot="R90">VCC</text>
+<text x="17.145" y="4.064" size="1.27" layer="21" font="vector" ratio="15" rot="R90">SDA</text>
+<text x="19.685" y="4.191" size="1.27" layer="21" font="vector" ratio="15" rot="R90">SCK</text>
+<text x="22.098" y="4.318" size="1.27" layer="21" font="vector" ratio="15" rot="R90">MOSI</text>
+<text x="24.765" y="4.191" size="1.27" layer="21" font="vector" ratio="15" rot="R90">MISO</text>
+<text x="32.385" y="4.191" size="1.27" layer="21" font="vector" ratio="15" rot="R90">RST</text>
+<text x="27.178" y="4.191" size="1.27" layer="21" font="vector" ratio="15" rot="R90">IRQ</text>
 <text x="0.508" y="31.242" size="1.27" layer="21" font="vector" ratio="15">PWR_IN</text>
 <text x="3.937" y="32.385" size="1.778" layer="21" font="vector" ratio="15">+</text>
 <text x="3.048" y="7.239" size="1.27" layer="21" font="vector" ratio="15">S'NOID/RLY</text>
 <text x="16.51" y="33.909" size="1.27" layer="21" font="vector" ratio="15">I2C</text>
-<text x="14.859" y="0.635" size="1.27" layer="21" font="vector" ratio="15">Access Controller V1.2</text>
+<text x="16.129" y="10.795" size="1.27" layer="21" font="vector" ratio="15">Access Controller</text>
 <text x="1.27" y="22.86" size="1.27" layer="21" font="vector" ratio="15" rot="R270">davidmpye@gmail.com</text>
 <text x="10.414" y="32.258" size="1.27" layer="21" font="vector" ratio="15">SDA</text>
@@
 <text x="10.668" y="34.544" size="1.27" layer="21" font="vector" ratio="15">3v3</text>
 <text x="10.414" y="37.465" size="1.27" layer="21" font="vector" ratio="15">GND</text>
-<text x="29.845" y="9.398" size="1.27" layer="21" font="vector" ratio="15" rot="R90">GND</text>
+<text x="29.845" y="4.318" size="1.27" layer="21" font="vector" ratio="15" rot="R90">GND</text>
 <text x="4.572" y="14.605" size="1.27" layer="21" font="vector" ratio="15">JP1</text>
+<text x="22.86" y="8.89" size="1.27" layer="21" font="vector" ratio="15">v1.2</text>
+<text x="2.921" y="12.319" size="0.8128" layer="21" font="vector">V_EXT</text>
+<text x="8.001" y="12.319" size="0.8128" layer="21" font="vector">V_3.3</text>
 </plain>
 <attributes>
@@
 </element>
 <element name="RELAY_HEADER" library="SparkFun-Connectors" package="1X03" value="" x="9.525" y="10.16" rot="R180"/>
-<element name="RFID_CONN" library="SparkFun-Connectors" package="1X08_ROUND" value="" x="16.51" y="6.35"/>
+<element name="RFID_CONN" library="SparkFun-Connectors" package="1X08_ROUND" value="" x="16.51" y="2.54"/>
 <element name="X1" library="adafruit" package="ESP-12" value="" x="31.115" y="26.035"/>
 <element name="PWR" library="SparkFun-Connectors" package="1X02" value="" x="2.54" y="36.449" rot="R270"/>
@@
 <wire x1="23.615" y1="16.535" x2="30.455" y2="16.535" width="0.4064" layer="1"/>
 <wire x1="30.455" y1="16.535" x2="34.29" y2="12.7" width="0.4064" layer="1"/>
-<wire x1="34.29" y1="12.7" x2="34.29" y2="6.35" width="0.4064" layer="1"/>
-<wire x1="48.26" y1="10.16" x2="38.1" y2="10.16" width="0.4064" layer="1"/>
-<wire x1="38.1" y1="10.16" x2="34.29" y2="6.35" width="0.4064" layer="1"/>
+<wire x1="34.29" y1="12.7" x2="34.29" y2="10.16" width="0.4064" layer="1"/>
+<wire x1="34.29" y1="10.16" x2="34.29" y2="2.54" width="0.4064" layer="1"/>
 <wire x1="48.26" y1="10.16" x2="46.99" y2="10.16" width="0.4064" layer="16"/>
 <wire x1="46.99" y1="10.16" x2="45.72" y2="11.43" width="0.4064" layer="16"/>
@@
 <wire x1="45.72" y1="20.32" x2="45.72" y2="19.05" width="0.4064" layer="16"/>
 <wire x1="45.72" y1="19.05" x2="48.26" y2="16.51" width="0.4064" layer="16"/>
+<wire x1="48.26" y1="10.16" x2="34.29" y2="10.16" width="0.4064" layer="1"/>
 </signal>
 <signal name="DTR">
@@
 <contactref element="RFID_CONN" pad="1"/>
 <contactref element="X1" pad="11"/>
-<wire x1="16.51" y1="6.35" x2="16.51" y2="10.16" width="0.4064" layer="1"/>
+<wire x1="16.51" y1="2.54" x2="16.51" y2="10.16" width="0.4064" layer="1"/>
 <via x="16.51" y="10.16" extent="1-16" drill="0.508"/>
 <wire x1="16.51" y1="10.16" x2="33.02" y2="10.16" width="0.4064" layer="16"/>
@@
 <signal name="RFID_MOSI">
 <contactref element="RFID_CONN" pad="3"/>
-<wire x1="21.59" y1="6.35" x2="21.59" y2="13.97" width="0.4064" layer="1"/>
+<wire x1="21.59" y1="2.54" x2="21.59" y2="13.97" width="0.4064" layer="1"/>
 <via x="21.59" y="13.97" extent="1-16" drill="0.508"/>
 <wire x1="21.59" y1="13.97" x2="21.59" y2="17.78" width="0.4064" layer="16"/>
@@
 <wire x1="25.4" y1="20.32" x2="23.4" y2="20.32" width="0.4064" layer="1"/>
 <wire x1="23.4" y1="20.32" x2="23.615" y2="20.535" width="0.4064" layer="1"/>
-<wire x1="24.13" y1="6.35" x2="24.13" y2="11.43" width="0.4064" layer="1"/>
+<wire x1="24.13" y1="2.54" x2="24.13" y2="11.43" width="0.4064" layer="1"/>
 <wire x1="24.13" y1="11.43" x2="25.4" y2="12.7" width="0.4064" layer="1"/>
 </signal>
@@
 <wire x1="31.75" y1="17.78" x2="31.75" y2="12.7" width="0.4064" layer="16"/>
 <via x="31.75" y="12.7" extent="1-16" drill="0.508"/>
-<wire x1="31.75" y1="12.7" x2="31.75" y2="6.35" width="0.4064" layer="1"/>
+<wire x1="31.75" y1="12.7" x2="31.75" y2="2.54" width="0.4064" layer="1"/>
 </signal>
 <signal name="RFID_SCK">
 <contactref element="RFID_CONN" pad="2"/>
 <contactref element="X1" pad="5"/>
-<wire x1="19.05" y1="6.35" x2="19.05" y2="15.24" width="0.4064" layer="1"/>
+<wire x1="19.05" y1="2.54" x2="19.05" y2="15.24" width="0.4064" layer="1"/>
 <via x="19.05" y="15.24" extent="1-16" drill="0.6"/>
 <wire x1="19.05" y1="15.24" x2="21.59" y2="21.59" width="0.4064" layer="16"/>
